File: 514_sensor_pcb/514_sensor_pcb.kicad_sch (KiCad schematic)
At the start: 3 parts

Commit message: Initial commit from workspace
Parts:
- removed U?: CR2032, symbol New_Library:CR2032
- added C1: C_Polarized_470uF, Capacitor_Tantalum_SMD:CP_EIA-6032-28_Kemet-C_HandSolder, symbol Device:C_Polarized_US
- added LIR2032: Battery 3.7V, Battery:BatteryHolder_Keystone_1057_1x2032, symbol Device:Battery
- U1: renamed from U; footprint XIAO_ESP32C3:xiao_esp32c3 -> RF_Module:MCU_Seeed_ESP32C3
- U2: renamed from U?; footprint (none) -> HTU21D:QFN100P300X300X100-7N
Connections:
- net GND: now reaches U1.13 (GND), U2.2 (GND), U2.7 (GND)
- net GND: now also U1.B- (Batt-), C1.2, LIR2032.2 (-)
- net VCC: now reaches U1.B+ (Batt+)
- net VCC: now also C1.1, LIR2032.1 (+)
Other:
- title: (none) -> YewenZhou_514sensor
- moved on the sheet: U1, U2
